Commit message: Add support namespace for multi robot configuration

File: former_description/urdf/former_ros2_control.urdf.xacro (robot description, xacro)
@@ -1,5 +1,5 @@
 <?xml version="1.0"?>
 <robot xmlns:xacro="http://www.ros.org/wiki/xacro">
-    <xacro:macro name="insert_ros2_control" params="name use_gazebo_sim:=^|false">
+    <xacro:macro name="insert_ros2_control" params="name prefix use_gazebo_sim:=^|false">
         <ros2_control name="${name}" type="system">
             <xacro:if value="$(arg use_gazebo_sim)">
@@ -17,5 +17,5 @@
                 </hardware>
             </xacro:unless>
-            <joint name="l_wheel_joint">
+            <joint name="${prefix}l_wheel_joint">
                 <command_interface name="velocity">
                     <param name="min">-1</param>
@@ -24,7 +24,7 @@
                 <state_interface name="position"/>
                 <state_interface name="velocity"/>
-                <!-- <state_interface name="effort"/> -->
+                <state_interface name="effort"/>
             </joint>
-            <joint name="r_wheel_joint">
+            <joint name="${prefix}r_wheel_joint">
                 <command_interface name="velocity">
                     <param name="min">-1</param>
@@ -33,8 +33,8 @@
                 <state_interface name="position"/>
                 <state_interface name="velocity"/>
-                <!-- <state_interface name="effort"/> -->
+                <state_interface name="effort"/>
             </joint>
             <xacro:unless value="$(arg use_gazebo_sim)">
-                <gpio name="gpio">
+                <gpio name="${prefix}gpio">
                     <command_interface name="set_enable_motor"/>
                     <state_interface name="motor_enabled"/>

File: former_description/urdf/robot.urdf.xacro (robot description, xacro)
@@ -1,5 +1,4 @@
 <?xml version="1.0"?>
 <robot xmlns:xacro="http://ros.org/wiki/xacro" name="former">
-    <xacro:arg name="use_gazebo_sim" default="false"/>
     <xacro:include filename="$(find former_description)/urdf/common/insert_inertia.urdf.xacro"/>
     <xacro:include filename="$(find former_description)/urdf/former.urdf.xacro"/>
@@ -7,5 +6,7 @@
     <xacro:include filename="$(find former_description)/urdf/former_ros2_control.urdf.xacro"/>
     <xacro:include filename="$(find realsense2_description)/urdf/_d435i.urdf.xacro"/>
-    <xacro:insert_robot prefix=""/>
-    <xacro:insert_ros2_control name="former_system" use_gazebo_sim="$(arg use_gazebo_sim)"/>
+    <xacro:arg name="use_gazebo_sim" default="false"/>
+    <xacro:arg name="tf_prefix" default=""/>
+    <xacro:insert_robot prefix="$(arg tf_prefix)"/>
+    <xacro:insert_ros2_control name="former_system" prefix="$(arg tf_prefix)" use_gazebo_sim="$(arg use_gazebo_sim)"/>
 </robot>

Commit message: add namespace for multi robot configuration

File: former_description/urdf/former_ros2_control.urdf.xacro (robot description, xacro)
@@ -17,5 +17,5 @@
                 </hardware>
             </xacro:unless>
-            <joint name="${prefix}l_wheel_joint">
+            <joint name="l_wheel_joint">
                 <command_interface name="velocity">
                     <param name="min">-1</param>
@@ -26,5 +26,5 @@
                 <state_interface name="effort"/>
             </joint>
-            <joint name="${prefix}r_wheel_joint">
+            <joint name="r_wheel_joint">
                 <command_interface name="velocity">
                     <param name="min">-1</param>
@@ -36,5 +36,5 @@
             </joint>
             <xacro:unless value="$(arg use_gazebo_sim)">
-                <gpio name="${prefix}gpio">
+                <gpio name="gpio">
                     <command_interface name="set_enable_motor"/>
                     <state_interface name="motor_enabled"/>
