Commit message: Add meshes and urdf files

File: former_description/urdf/former.urdf.xacro (robot description, xacro)
@@ -4,6 +4,6 @@
         <xacro:property name="wheel_radius" value="0.159"/>
         <xacro:property name="wheel_seperation" value="0.4"/>
-        <link name="base_footprint"/>
-        <link name="base_link">
+        <link name="${prefix}base_footprint"/>
+        <link name="${prefix}base_link">
             <visual>
                 <origin xyz="0 0 0" rpy="0 0 0"/>
@@ -24,10 +24,34 @@
             </inertial>
         </link>
-        <joint name="base_link_fixed_joint" type="fixed">
-            <parent link="base_footprint"/>
-            <child link="base_link"/>
-            <origin xyz="0 0 0.08" rpy="0 0 0"/>
+        <joint name="${prefix}base_link_fixed_joint" type="fixed">
+            <parent link="${prefix}base_footprint"/>
+            <child link="${prefix}base_link"/>
+            <origin xyz="0 0 ${0.169/2}" rpy="0 0 0"/>
         </joint>
-        <!-- <xacro:macro name="insert_wheel" params="prefix dir">
+        <xacro:macro name="insert_wheel" params="parent prefix dir">
+            <link name="${prefix}_wheel_mount">
+                <visual>
+                    <origin xyz="0 0 0" rpy="0 0 ${dir*pi/2}"/>
+                    <geometry>
+                        <mesh filename="package://former_description/meshes/visual/main_wheel_mount.dae" scale="1 1 1"/>
+                    </geometry>
+                </visual>
+                <collision>
+                    <origin xyz="0 0 0" rpy="0 0 ${dir*pi/2}"/>
+                    <geometry>
+                        <mesh filename="package://former_description/meshes/collision/main_wheel_mount.stl" scale="1 1 1"/>
+                    </geometry>
+                </collision>
+                <inertial>
+                    <origin xyz="0 0 0" rpy="0 0 ${dir*pi/2}"/>
+                    <mass value="67.084"/>
+                    <inertia ixx="1.067955" ixy="0.010608" ixz="-0.044928" iyy="2.497383" iyz="-0.000028" izz="3.217104"/>
+                </inertial>
+            </link>
+            <joint name="${prefix}_wheel_mount_fixed" type="fixed">
+                <parent link="${parent}"/>
+                <child link="${prefix}_wheel_mount"/>
+                <origin xyz="0 ${dir*0.0711} 0" rpy="0 0 0"/>
+            </joint>
             <link name="${prefix}_wheel">
                 <visual>
@@ -38,11 +62,12 @@
                 </visual>
                 <collision>
-                    <origin xyz="0 ${dir*-0.011} 0.0" rpy="${pi/2} 0 0"/>
-                    <geometry>
-                        <cylinder radius="0.08" length="0.05"/>
-                    </geometry>
-                </collision>
-                <inertial>
-                    <origin xyz="0 ${dir*-0.011} 0.0" rpy="${pi/2} 0 0"/>
+                    <origin xyz="0 0 0" rpy="0 0 ${dir*pi/2}"/>
+                    <geometry>
+                        <!-- <cylinder radius="0.08" length="0.05"/> -->
+                        <mesh filename="package://former_description/meshes/collision/main_wheel.stl" scale="1 1 1"/>
+                    </geometry>
+                </collision>
+                <inertial>
+                    <origin xyz="0 0 0" rpy="0 0 ${dir*pi/2}"/>
                     <mass value="0.323442"/>
                     <xacro:cylinder_inertia m="0.323442" r="0.08" h="0.05"/>
@@ -50,13 +75,155 @@
             </link>
             <joint name="${prefix}_wheel_joint" type="continuous">
-                <parent link="base_link"/>
+                <parent link="${prefix}_wheel_mount"/>
                 <child link="${prefix}_wheel"/>
                 <axis xyz="0 1 0"/>
-                <origin xyz="0 ${dir*0.246} 0" rpy="0 0 0"/>
+                <origin xyz="0 ${dir*0.051} 0" rpy="0 0 0"/>
             </joint>
             <xacro:insert_velocity_transmission name="${prefix}_wheel_joint"/>
         </xacro:macro>
-        <xacro:insert_wheel prefix="l" dir="1"/>
-        <xacro:insert_wheel prefix="r" dir="-1"/> -->
+        <xacro:insert_wheel parent="${prefix}base_link" prefix="${prefix}l" dir="1" />
+        <xacro:insert_wheel parent="${prefix}base_link" prefix="${prefix}r" dir="-1" />
+        <xacro:macro name="insert_front_caster_wheel" params="parent prefix1 prefix2 dir offset_x offset_y">
+            <link name="${prefix1}_${prefix2}_caster_mount">
+                <visual>
+                    <origin xyz="0 0 0" rpy="0 0 0"/>
+                    <geometry>
+                        <mesh filename="package://former_description/meshes/visual/caster_mount.dae" scale="1 1 1"/>
+                    </geometry>
+                </visual>
+                <collision>
+                    <origin xyz="0 0 0" rpy="0 0 0"/>
+                    <geometry>
+                        <mesh filename="package://former_description/meshes/collision/caster_mount.stl" scale="1 1 1"/>
+                    </geometry>
+                </collision>
+                <inertial>
+                    <origin xyz="0.000 0.000 -0.007" rpy="0 0 0"/>
+                    <mass value="0.042084"/>
+                    <inertia ixx="0.000030" ixy="0.0" ixz="0.0" iyy="0.000030" iyz="0.0" izz="0.000059"/>
+                </inertial>
+            </link>
+            <joint name="${prefix1}_${prefix2}_caster_mount_fixed_joint" type="fixed">
+                <parent link="${parent}"/>
+                <child link="${prefix1}_${prefix2}_caster_mount"/>
+                <origin xyz="${offset_x} ${dir*offset_y} -0.0015" rpy="0 0 0"/>
+            </joint>
+            <link name="${prefix1}_${prefix2}_caster_rotate">
+                <visual>
+                    <origin xyz="0 0 0" rpy="0 0 0"/>
+                    <geometry>
+                        <mesh filename="package://former_description/meshes/visual/caster_rotate.dae" scale="1 1 1"/>
+                    </geometry>
+                </visual>
+                <collision>
+                    <origin xyz="0 0 0" rpy="0 0 0"/>
+                    <geometry>
+                        <mesh filename="package://former_description/meshes/collision/caster_rotate.stl" scale="1 1 1"/>
+                    </geometry>
+                </collision>
+                <inertial>
+                    <origin xyz="-0.016 0.000 -0.034" rpy="0 0 0"/>
+                    <mass value="0.106803"/>
+                    <inertia ixx="0.000088" ixy="0.0" ixz="-0.000017" iyy="0.000085" iyz="0.0" izz="0.000093"/>
+                </inertial>
+            </link>
+            <joint name="${prefix1}_${prefix2}_caster_rotate_joint" type="continuous">
+                <parent link="${prefix1}_${prefix2}_caster_mount"/>
+                <child link="${prefix1}_${prefix2}_caster_rotate"/>
+                <axis xyz="0 0 1"/>
+                <origin xyz="0 0 -0.010" rpy="0 0 0"/>
+            </joint>
+            <link name="${prefix1}_${prefix2}_caster_wheel">
+                <visual>
+                    <origin xyz="0 0 0" rpy="0 0 0"/>
+                    <geometry>
+                        <mesh filename="package://former_description/meshes/visual/caster_wheel.dae" scale="1 1 1"/>
+                    </geometry>
+                </visual>
+                <collision>
+                    <origin xyz="0 0 0" rpy="0 0 0"/>
+                    <geometry>
+                        <mesh filename="package://former_description/meshes/collision/caster_wheel.stl" scale="1 1 1"/>
+                        <!-- <cylinder radius="0.0375" length="0.023"/> -->
+                    </geometry>
+                </collision>
+                <inertial>
+                    <origin xyz="0 0 0" rpy="0 0 0"/>
+                    <mass value="0.032222"/>
+                    <xacro:cylinder_inertia m="0.032222" r="0.0375" h="0.023"/>
+                </inertial>
+            </link>
+            <joint name="${prefix1}_${prefix2}_caster_wheel_joint" type="continuous">
+                <parent link="${prefix1}_${prefix2}_caster_rotate"/>
+                <child link="${prefix1}_${prefix2}_caster_wheel"/>
+                <axis xyz="0 1 0"/>
+                <origin xyz="-0.0235 0 -0.0415" rpy="0 0 0"/>
+            </joint>
+        </xacro:macro>
+        <xacro:insert_front_caster_wheel parent="${prefix}base_link" prefix1="${prefix}f" prefix2="l" dir="1" offset_x="0.125" offset_y="0.087"/>
+        <xacro:insert_front_caster_wheel parent="${prefix}base_link" prefix1="${prefix}f" prefix2="r" dir="-1" offset_x="0.125" offset_y="0.087"/>
+        <xacro:insert_front_caster_wheel parent="${prefix}base_link" prefix1="${prefix}r" prefix2="l" dir="1" offset_x="-0.128" offset_y="0.099"/>
+        <xacro:insert_front_caster_wheel parent="${prefix}base_link" prefix1="${prefix}r" prefix2="r" dir="-1" offset_x="-0.128" offset_y="0.099"/>
+        <xacro:macro name="insert_sonar_sensor" params="parent prefix dir">
+            <link name="${prefix}_sonar_sensor">
+                <visual>
+                        <origin xyz="0 0 0" rpy="0 0 0"/>
+                        <geometry>
+                            <mesh filename="package://former_description/meshes/visual/sonar_sensor.dae" scale="1 1 1"/>
+                        </geometry>
+                    </visual>
+                    <collision>
+                        <origin xyz="0 0 0" rpy="0 0 0"/>
+                        <geometry>
+                            <mesh filename="package://former_description/meshes/collision/sonar_sensor.stl" scale="1 1 1"/>
+                        </geometry>
+                    </collision>
+                    <inertial>
+                        <origin xyz="0 0 0" rpy="0 0 0"/>
+                        <mass value="0.032222"/>
+                        <xacro:cylinder_inertia m="0.032222" r="0.0375" h="0.023"/>
+                    </inertial>
+            </link>
+            <joint name="${prefix}_sonar_sensor_fixed" type="fixed">
+                <parent link="${parent}"/>
+                <child link="${prefix}_sonar_sensor"/>
+                <origin xyz="0.184 ${dir*0.0968} 0.084" rpy="0 0 0"/>
+            </joint>
+        </xacro:macro>
+        <xacro:insert_sonar_sensor parent="${prefix}base_link" prefix="${prefix}l" dir="1" />
+        <xacro:insert_sonar_sensor parent="${prefix}base_link" prefix="${prefix}r" dir="-1" />
+        <link name="${prefix}lidar_mount">
+            <visual>
+                <origin xyz="0 0 0" rpy="0 0 0"/>
+                <geometry>
+                    <mesh filename="package://former_description/meshes/visual/sick_tim5_lidar.dae" scale="1 1 1"/>
+                </geometry>
+            </visual>
+            <collision>
+                <origin xyz="0 0 0" rpy="0 0 0"/>
+                <geometry>
+                    <mesh filename="package://former_description/meshes/collision/sick_tim5_lidar.stl" scale="1 1 1"/>
+                </geometry>
+            </collision>
+            <inertial>
+                <origin xyz="0.010 0.000 0.070" rpy="0 0 0"/>
+                <mass value="67.084"/>
+                <inertia ixx="1.067955" ixy="0.010608" ixz="-0.044928" iyy="2.497383" iyz="-0.000028" izz="3.217104"/>
+            </inertial>
+        </link>
+        <joint name="${prefix}lidar_mount_fixed_joint" type="fixed">
+            <parent link="${prefix}base_link"/>
+            <child link="${prefix}lidar_mount"/>
+            <origin xyz="0.160 0 0.2275" rpy="${pi} 0 0"/>
+        </joint>
+        <link name="${prefix}laser_link"/>
+        <joint name="${prefix}laser_link_fixed_joint" type="fixed">
+            <parent link="${prefix}lidar_mount"/>
+            <child link="${prefix}laser_link"/>
+            <origin xyz="0 0 0.060" rpy="${pi} 0 0"/>
+        </joint>
+        <xacro:sensor_d435i parent="${prefix}base_link" name="${prefix}camera" use_nominal_extrinsics="false">
+            <origin xyz="0.1777 0 0.06715" rpy="0 ${-15*pi/180} 0"/>
+        </xacro:sensor_d435i>
     </xacro:macro>
 </robot>

File: former_description/urdf/robot.urdf.xacro (robot description, xacro)
@@ -5,4 +5,5 @@
     <xacro:include filename="$(find former_description)/urdf/common/insert_transmission.urdf.xacro"/>
     <xacro:include filename="$(find former_description)/urdf/former.urdf.xacro"/>
+    <xacro:include filename="$(find realsense2_description)/urdf/_d435i.urdf.xacro"/>
     <xacro:insert_robot prefix="$(arg prefix)"/>
 </robot>

Commit message: Add inertia for link and sensors

File: former_description/urdf/former.urdf.xacro (robot description, xacro)
@@ -19,7 +19,7 @@
             </collision>
             <inertial>
-                <origin xyz="0.010 0.000 0.070" rpy="0 0 0"/>
-                <mass value="67.084"/>
-                <inertia ixx="1.067955" ixy="0.010608" ixz="-0.044928" iyy="2.497383" iyz="-0.000028" izz="3.217104"/>
+                <origin xyz="0.000 0.000 0.096" rpy="0 0 0"/>
+                <mass value="32.571233"/>
+                <inertia ixx="0.639569" ixy="0.000014" ixz="0.000423" iyy="0.635798" iyz="0.000003" izz="0.798308"/>
             </inertial>
         </link>
@@ -44,7 +44,7 @@
                 </collision>
                 <inertial>
-                    <origin xyz="0 0 0" rpy="0 0 ${dir*pi/2}"/>
-                    <mass value="67.084"/>
-                    <inertia ixx="1.067955" ixy="0.010608" ixz="-0.044928" iyy="2.497383" iyz="-0.000028" izz="3.217104"/>
+                    <origin xyz="0.026 0.000 0.000" rpy="0 0 ${dir*pi/2}"/>
+                    <mass value="0.007885"/>
+                    <inertia ixx="0.000000" ixy="0.000000" ixz="0.000000" iyy="0.000002" iyz="0.000000" izz="0.000002"/>
                 </inertial>
             </link>
@@ -69,7 +69,8 @@
                 </collision>
                 <inertial>
-                    <origin xyz="0 0 0" rpy="0 0 ${dir*pi/2}"/>
-                    <mass value="0.323442"/>
-                    <xacro:cylinder_inertia m="0.323442" r="0.08" h="0.05"/>
+                    <origin xyz="0.000 ${dir*0.031} 0.000" rpy="0 0 ${dir*pi/2}"/>
+                    <mass value="0.843041"/>
+                    <!-- <xacro:cylinder_inertia m="0.323442" r="0.08" h="0.05"/> -->
+                    <inertia ixx="0.002632" ixy="0.000000" ixz="0.000000" iyy="0.001536" iyz="0.000000" izz="0.001536"/>
                 </inertial>
             </link>
@@ -99,7 +100,7 @@
                 </collision>
                 <inertial>
-                    <origin xyz="0.000 0.000 -0.007" rpy="0 0 0"/>
-                    <mass value="0.042084"/>
-                    <inertia ixx="0.000030" ixy="0.0" ixz="0.0" iyy="0.000030" iyz="0.0" izz="0.000059"/>
+                    <origin xyz="0.000 0.000 -0.004" rpy="0 0 0"/>
+                    <mass value="0.019629"/>
+                    <inertia ixx="0.000006" ixy="0.000000" ixz="0.000000" iyy="0.000005" iyz="0.000000" izz="0.000010"/>
                 </inertial>
             </link>
@@ -123,7 +124,7 @@
                 </collision>
                 <inertial>
-                    <origin xyz="-0.016 0.000 -0.034" rpy="0 0 0"/>
-                    <mass value="0.106803"/>
-                    <inertia ixx="0.000088" ixy="0.0" ixz="-0.000017" iyy="0.000085" iyz="0.0" izz="0.000093"/>
+                    <origin xyz="-0.012 0.000 -0.021" rpy="0 0 0"/>
+                    <mass value="0.060591"/>
+                    <inertia ixx="0.000020" ixy="0.000000" ixz="-0.000004" iyy="0.000022" iyz="0.000000" izz="0.000020"/>
                 </inertial>
             </link>
@@ -149,7 +150,8 @@
                 </collision>
                 <inertial>
-                    <origin xyz="0 0 0" rpy="0 0 0"/>
-                    <mass value="0.032222"/>
-                    <xacro:cylinder_inertia m="0.032222" r="0.0375" h="0.023"/>
+                    <origin xyz="0.000 0.000 0.000" rpy="0 0 0"/>
+                    <mass value="0.051842"/>
+                    <!-- <xacro:cylinder_inertia m="0.032222" r="0.0375" h="0.023"/> -->
+                    <inertia ixx="0.000013" ixy="0.000000" ixz="0.000000" iyy="0.000021" iyz="0.000000" izz="0.000013"/>
                 </inertial>
             </link>
@@ -180,7 +182,7 @@
                     </collision>
                     <inertial>
-                        <origin xyz="0 0 0" rpy="0 0 0"/>
-                        <mass value="0.032222"/>
-                        <xacro:cylinder_inertia m="0.032222" r="0.0375" h="0.023"/>
+                        <origin xyz="0.004 0.002 0.000" rpy="0 0 0"/>
+                        <mass value="0.009290"/>
+                        <inertia ixx="0.000001" ixy="0.000000" ixz="0.000000" iyy="0.000001" iyz="0.000000" izz="0.000001"/>
                     </inertial>
             </link>
@@ -207,7 +209,7 @@
             </collision>
             <inertial>
-                <origin xyz="0.010 0.000 0.070" rpy="0 0 0"/>
-                <mass value="67.084"/>
-                <inertia ixx="1.067955" ixy="0.010608" ixz="-0.044928" iyy="2.497383" iyz="-0.000028" izz="3.217104"/>
+                <origin xyz="-0.002 0.000 0.036" rpy="0 0 0"/>
+                <mass value="0.180090"/>
+                <inertia ixx="0.000139" ixy="0.000000" ixz="0.000002" iyy="0.000129" iyz="0.000000" izz="0.000094"/>
             </inertial>
         </link>

File: former_description/urdf/robot.urdf.xacro (robot description, xacro)
@@ -5,4 +5,5 @@
     <xacro:include filename="$(find former_description)/urdf/common/insert_transmission.urdf.xacro"/>
     <xacro:include filename="$(find former_description)/urdf/former.urdf.xacro"/>
+    <xacro:include filename="$(find former_description)/urdf/former_gazebo.urdf.xacro"/>
     <xacro:include filename="$(find realsense2_description)/urdf/_d435i.urdf.xacro"/>
     <xacro:insert_robot prefix="$(arg prefix)"/>

Commit message: add simulation package for gazebo

File: former_description/urdf/former.urdf.xacro (robot description, xacro)
@@ -62,15 +62,17 @@
                 </visual>
                 <collision>
-                    <origin xyz="0 0 0" rpy="0 0 ${dir*pi/2}"/>
-                    <geometry>
-                        <!-- <cylinder radius="0.08" length="0.05"/> -->
-                        <mesh filename="package://former_description/meshes/collision/main_wheel.stl" scale="1 1 1"/>
-                    </geometry>
-                </collision>
-                <inertial>
-                    <origin xyz="0.000 ${dir*0.031} 0.000" rpy="0 0 ${dir*pi/2}"/>
+                    <origin xyz="0 ${dir*0.025} 0" rpy="${dir*pi/2} 0 0"/>
+                    <!-- <origin xyz="0 0 0" rpy="0 0 ${dir*pi/2}"/> -->
+                    <geometry>
+                        <cylinder radius="0.0845" length="0.05"/>
+                        <!-- <mesh filename="package://former_description/meshes/collision/main_wheel.stl" scale="1 1 1"/> -->
+                    </geometry>
+                </collision>
+                <inertial>
+                    <origin xyz="0 ${dir*0.025} 0" rpy="${dir*pi/2} 0 0"/>
+                    <!-- <origin xyz="0.000 ${dir*0.031} 0.000" rpy="0 0 0"/> -->
                     <mass value="0.843041"/>
-                    <!-- <xacro:cylinder_inertia m="0.323442" r="0.08" h="0.05"/> -->
-                    <inertia ixx="0.002632" ixy="0.000000" ixz="0.000000" iyy="0.001536" iyz="0.000000" izz="0.001536"/>
+                    <xacro:cylinder_inertia m="0.843041" r="0.0845" h="0.05"/>
+                    <!-- <inertia ixx="0.002632" ixy="0.000000" ixz="0.000000" iyy="0.001536" iyz="0.000000" izz="0.001536"/> -->
                 </inertial>
             </link>

File: former_description/urdf/former_gazebo.urdf.xacro (robot description, xacro)
@@ -4,5 +4,5 @@
         <plugin filename="ign_ros2_control-system" name="ign_ros2_control::IgnitionROS2ControlPlugin">
             <robot_param>robot_description</robot_param>
-            <parameters>$(find former_bringup)/config/controllers_former.yaml</parameters>
+            <parameters>$(find former_bringup)/config/controllers_former_gazebo.yaml</parameters>
         </plugin>
         <plugin filename="ignition-gazebo-sensors-system" name="ignition::gazebo::systems::Sensors">
@@ -56,6 +56,6 @@
     </gazebo>
     <gazebo reference="laser_link">
-        <sensor name='laser_sensor' type='gpu_lidar'>
-            <topic>front_scan</topic>
+        <sensor name="laser_link" type="gpu_lidar">
+            <topic>laser_scan</topic>
             <update_rate>15</update_rate>
             <alwaysOn>1</alwaysOn>

File: former_description/urdf/former_ros2_control.urdf.xacro (robot description, xacro)
@@ -2,5 +2,5 @@
 <robot xmlns:xacro="http://www.ros.org/wiki/xacro">
     <xacro:macro name="insert_ros2_control" params="name use_gazebo_sim:=^|false">
-        <ros2_control name="name" type="system">
+        <ros2_control name="${name}" type="system">
             <xacro:if value="$(arg use_gazebo_sim)">
                 <hardware>
@@ -13,6 +13,6 @@
             <joint name="l_wheel_joint">
                 <command_interface name="velocity">
-                    <param name="min">-20.0</param>
-                    <param name="max">20.0</param>
+                    <param name="min">-1.0</param>
+                    <param name="max">1.0</param>
                 </command_interface>
                 <state_interface name="position"/>
@@ -21,6 +21,6 @@
             <joint name="r_wheel_joint">
                 <command_interface name="velocity">
-                    <param name="min">-20.0</param>
-                    <param name="max">20.0</param>
+                    <param name="min">-1.0</param>
+                    <param name="max">1.0</param>
                 </command_interface>
                 <state_interface name="position"/>
