Commit message: bug fixed

File: former_description/urdf/former.urdf.xacro (robot description, xacro)
@@ -2,5 +2,5 @@
 <robot xmlns:xacro="http://www.ros.org/wiki/xacro">
     <xacro:macro name="insert_robot" params="prefix">
-        <xacro:property name="wheel_radius" value="0.159"/>
+        <xacro:property name="wheel_radius" value="0.169"/>
         <xacro:property name="wheel_seperation" value="0.4"/>
         <link name="${prefix}base_footprint"/>
@@ -27,5 +27,5 @@
             <parent link="${prefix}base_footprint"/>
             <child link="${prefix}base_link"/>
-            <origin xyz="0 0 ${0.169/2}" rpy="0 0 0"/>
+            <origin xyz="0 0 ${wheel_radius/2}" rpy="0 0 0"/>
         </joint>
         <xacro:macro name="insert_wheel" params="parent prefix dir">
@@ -62,17 +62,17 @@
                 </visual>
                 <collision>
-                    <origin xyz="0 ${dir*0.025} 0" rpy="${dir*pi/2} 0 0"/>
-                    <!-- <origin xyz="0 0 0" rpy="0 0 ${dir*pi/2}"/> -->
-                    <geometry>
-                        <cylinder radius="0.0845" length="0.05"/>
-                        <!-- <mesh filename="package://former_description/meshes/collision/main_wheel.stl" scale="1 1 1"/> -->
-                    </geometry>
-                </collision>
-                <inertial>
-                    <origin xyz="0 ${dir*0.025} 0" rpy="${dir*pi/2} 0 0"/>
-                    <!-- <origin xyz="0.000 ${dir*0.031} 0.000" rpy="0 0 0"/> -->
+                    <!-- <origin xyz="0 ${dir*0.025} 0" rpy="${dir*pi/2} 0 0"/> -->
+                    <origin xyz="0 0 0" rpy="0 0 ${dir*pi/2}"/>
+                    <geometry>
+                        <!-- <cylinder radius="0.0845" length="0.05"/> -->
+                        <mesh filename="package://former_description/meshes/collision/main_wheel.stl" scale="1 1 1"/>
+                    </geometry>
+                </collision>
+                <inertial>
+                    <!-- <origin xyz="0 ${dir*0.025} 0" rpy="${dir*pi/2} 0 0"/> -->
+                    <origin xyz="0.000 ${dir*0.031} 0.000" rpy="0 0 0"/>
                     <mass value="0.843041"/>
-                    <xacro:cylinder_inertia m="0.843041" r="0.0845" h="0.05"/>
-                    <!-- <inertia ixx="0.002632" ixy="0.000000" ixz="0.000000" iyy="0.001536" iyz="0.000000" izz="0.001536"/> -->
+                    <!-- <xacro:cylinder_inertia m="0.843041" r="0.0845" h="0.05"/> -->
+                    <inertia ixx="0.002632" ixy="0.000000" ixz="0.000000" iyy="0.001536" iyz="0.000000" izz="0.001536"/>
                 </inertial>
             </link>

Commit message: Add IMU sensor

File: former_description/urdf/former.urdf.xacro (robot description, xacro)
@@ -168,23 +168,53 @@
         <xacro:insert_front_caster_wheel parent="${prefix}base_link" prefix1="${prefix}r" prefix2="l" dir="1" offset_x="-0.128" offset_y="0.099"/>
         <xacro:insert_front_caster_wheel parent="${prefix}base_link" prefix1="${prefix}r" prefix2="r" dir="-1" offset_x="-0.128" offset_y="0.099"/>
+        <link name="${prefix}imu_sensor">
+            <visual>
+                <origin xyz="0 0 0" rpy="0 0 0"/>
+                <geometry>
+                    <mesh filename="package://former_description/meshes/visual/imu.dae" scale="1 1 1"/>
+                </geometry>
+            </visual>
+            <collision>
+                <origin xyz="0 0 0" rpy="0 0 0"/>
+                <geometry>
+                    <mesh filename="package://former_description/meshes/collision/imu.stl" scale="1 1 1"/>
+                </geometry>
+            </collision>
+            <inertial>
+                <origin xyz="0.0 0.0 0.0045" rpy="0 0 0"/>
+                <mass value="0.1"/>
+                <xacro:box_inertia m="0.032" x="0.032" y="0.032" z="0.009"/>
+            </inertial>
+        </link>
+        <joint name="${prefix}imu_sensor_fixed_joint" type="fixed">
+            <parent link="${prefix}base_link"/>
+            <child link="${prefix}imu_sensor"/>
+            <origin xyz="0.134 0 0.0045" rpy="0 0 0"/>
+        </joint>
+        <link name="${prefix}imu_link"/>
+        <joint name="${prefix}imu_link_fixed_joint" type="fixed">
+            <parent link="${prefix}imu_sensor"/>
+            <child link="${prefix}imu_link"/>
+            <origin xyz="0.0 0.0 0.009"/>
+        </joint>
         <xacro:macro name="insert_sonar_sensor" params="parent prefix dir">
             <link name="${prefix}_sonar_sensor">
                 <visual>
-                        <origin xyz="0 0 0" rpy="0 0 0"/>
-                        <geometry>
-                            <mesh filename="package://former_description/meshes/visual/sonar_sensor.dae" scale="1 1 1"/>
-                        </geometry>
-                    </visual>
-                    <collision>
-                        <origin xyz="0 0 0" rpy="0 0 0"/>
-                        <geometry>
-                            <mesh filename="package://former_description/meshes/collision/sonar_sensor.stl" scale="1 1 1"/>
-                        </geometry>
-                    </collision>
-                    <inertial>
-                        <origin xyz="0.004 0.002 0.000" rpy="0 0 0"/>
-                        <mass value="0.009290"/>
-                        <inertia ixx="0.000001" ixy="0.000000" ixz="0.000000" iyy="0.000001" iyz="0.000000" izz="0.000001"/>
-                    </inertial>
+                    <origin xyz="0 0 0" rpy="0 0 0"/>
+                    <geometry>
+                        <mesh filename="package://former_description/meshes/visual/sonar_sensor.dae" scale="1 1 1"/>
+                    </geometry>
+                </visual>
+                <collision>
+                    <origin xyz="0 0 0" rpy="0 0 0"/>
+                    <geometry>
+                        <mesh filename="package://former_description/meshes/collision/sonar_sensor.stl" scale="1 1 1"/>
+                    </geometry>
+                </collision>
+                <inertial>
+                    <origin xyz="0.004 0.002 0.000" rpy="0 0 0"/>
+                    <mass value="0.009290"/>
+                    <inertia ixx="0.000001" ixy="0.000000" ixz="0.000000" iyy="0.000001" iyz="0.000000" izz="0.000001"/>
+                </inertial>
             </link>
             <joint name="${prefix}_sonar_sensor_fixed" type="fixed">

File: former_description/urdf/former_gazebo.urdf.xacro (robot description, xacro)
@@ -8,4 +8,6 @@
         <plugin filename="ignition-gazebo-sensors-system" name="ignition::gazebo::systems::Sensors">
             <render_engine>ogre2</render_engine>
+        </plugin>
+        <plugin filename="ignition-gazebo-imu-system" name="ignition::gazebo::systems::Imu">
         </plugin>
     </gazebo>
@@ -89,3 +91,37 @@
         </sensor>
     </gazebo>
+    <gazebo reference="imu_link">
+        <sensor name="imu" type="imu">
+            <always_on>1</always_on>
+            <update_rate>100</update_rate>
+            <visualize>true</visualize>
+            <topic>imu</topic>
+            <enable_metrics>true</enable_metrics>
+        </sensor>
+    </gazebo>
+    <gazebo reference="camera_link">
+        <sensor name="rgbd_camera" type="rgbd_camera">
+            <always_on>1</always_on>
+            <update_rate>30</update_rate>
+            <visualize>true</visualize>
+            <topic>camera</topic>
+            <enable_metrics>true</enable_metrics>
+            <camera>
+                <horizontal_fov>1.047</horizontal_fov>
+                <image>
+                    <width>640</width>
+                    <height>480</height>
+                </image>
+                <clip>
+                    <near>0.1</near>
+                    <far>100</far>
+                </clip>
+            </camera>
+            <noise>
+                <type>gaussian</type>
+                <mean>0.0</mean>
+                <stddev>0.02</stddev>
+            </noise>
+        </sensor>
+    </gazebo>
 </robot>

Commit message: add ros2_controllers

File: former_description/urdf/former.urdf.xacro (robot description, xacro)
@@ -71,5 +71,5 @@
                 <inertial>
                     <!-- <origin xyz="0 ${dir*0.025} 0" rpy="${dir*pi/2} 0 0"/> -->
-                    <origin xyz="0.000 ${dir*0.031} 0.000" rpy="0 0 0"/>
+                    <origin xyz="0.000 ${dir*0.031} 0.000" rpy="0 0 ${dir*pi/2}"/>
                     <mass value="0.843041"/>
                     <!-- <xacro:cylinder_inertia m="0.843041" r="0.0845" h="0.05"/> -->
@@ -259,4 +259,10 @@
             <origin xyz="0.1777 0 0.06715" rpy="0 ${-15*pi/180} 0"/>
         </xacro:sensor_d435i>
+        <link name="${prefix}camera_depth_frame"/>
+        <joint name="${prefix}camera_depth_frame_fixed" type="fixed">
+            <parent link="${prefix}camera_link"/>
+            <child link="${prefix}camera_depth_frame"/>
+            <origin xyz="0 0 0" rpy="${-pi/2} 0 ${-pi/2}"/>
+        </joint>
     </xacro:macro>
 </robot>

File: former_description/urdf/former_gazebo.urdf.xacro (robot description, xacro)
@@ -1,15 +1,9 @@
 <?xml version="1.0"?>
 <robot xmlns:xacro="http://www.ros.org/wiki/xacro">
-    <!-- <gazebo>
-        <plugin filename="gz_ros2_control-system" name="gz_ros2_control::GazeboSimROS2ControlPlugin">
-            <robot_param>robot_description</robot_param>
-            <parameters>$(find former_bringup)/config/controllers_former_gazebo.yaml</parameters>
+    <gazebo>
+        <plugin filename="libgazebo_ros2_control.so" name="gazebo_ros2_control">
+        <parameters>$(find former_bringup)/config/controllers_former_gazebo.yaml</parameters>
         </plugin>
-        <plugin filename="gz-sim-sensors-system" name="gz::sim::systems::Sensors">
-            <render_engine>ogre2</render_engine>
-        </plugin>
-        <plugin filename="gz-sim-imu-system" name="gz::sim::systems::Imu">
-        </plugin>
-    </gazebo> -->
+    </gazebo>
     <gazebo reference="l_wheel">
         <mu1>200</mu1>
@@ -27,5 +21,19 @@
     </gazebo>
     <gazebo reference="f_l_caster_wheel">
-        <mu1>1</mu1>
+        <mu1>0.1</mu1>
+        <mu2>0.1</mu2>
+        <kp>10000000.0</kp>
+        <kd>1.0</kd>
+        <!-- <minDepth>0.001</minDepth> -->
+    </gazebo>
+    <gazebo reference="f_r_caster_wheel">
+        <mu1>0.1</mu1>
+        <mu2>0.1</mu2>
+        <kp>10000000.0</kp>
+        <kd>1.0</kd>
+        <!-- <minDepth>0.001</minDepth> -->
+    </gazebo>
+    <gazebo reference="r_l_caster_wheel">
+        <mu1>0.1</mu1>
         <mu2>1</mu2>
         <kp>10000000.0</kp>
@@ -33,21 +41,7 @@
         <!-- <minDepth>0.001</minDepth> -->
     </gazebo>
-    <gazebo reference="f_r_caster_wheel">
-        <mu1>1</mu1>
-        <mu2>1</mu2>
-        <kp>10000000.0</kp>
-        <kd>1.0</kd>
-        <!-- <minDepth>0.001</minDepth> -->
-    </gazebo>
-    <gazebo reference="r_l_caster_wheel">
-        <mu1>1</mu1>
-        <mu2>1</mu2>
-        <kp>10000000.0</kp>
-        <kd>1.0</kd>
-        <!-- <minDepth>0.001</minDepth> -->
-    </gazebo>
     <gazebo reference="r_r_caster_wheel">
-        <mu1>1</mu1>
-        <mu2>1</mu2>
+        <mu1>0.1</mu1>
+        <mu2>0.1</mu2>
         <kp>10000000.0</kp>
         <kd>1.0</kd>
@@ -57,28 +51,22 @@
         <self_collide>0</self_collide>
     </gazebo>
-    <!-- <gazebo reference="laser_link">
-        <sensor name="laser_link" type="gpu_lidar">
-            <topic>scan</topic>
+    <gazebo reference="laser_link">
+        <sensor name="laser" type="ray">
+            <pose>0 0 0 0 0 0</pose>
+            <always_on>1</always_on>
             <update_rate>15</update_rate>
-            <alwaysOn>1</alwaysOn>
-            <visualize>true</visualize>
-            <lidar>
+            <visualize>true</visualize>
+            <ray>
                 <scan>
                     <horizontal>
                         <samples>640</samples>
                         <resolution>1</resolution>
-                        <min_angle>${-110/180*pi}</min_angle>
-                        <max_angle>${110/180*pi}</max_angle>
+                        <min_angle>-1.26889</min_angle>
+                        <max_angle>1.268899</max_angle>
                     </horizontal>
-                    <vertical>
-                        <samples>1</samples>
-                        <resolution>0.01</resolution>
-                        <min_angle>0</min_angle>
-                        <max_angle>0</max_angle>
-                    </vertical>
                 </scan>
                 <range>
-                    <min>0.08</min>
-                    <max>15.0</max>
+                    <min>0.1</min>
+                    <max>15</max>
                     <resolution>0.01</resolution>
                 </range>
@@ -86,44 +74,116 @@
                     <type>gaussian</type>
                     <mean>0.0</mean>
-                    <stddev>0.02</stddev>
+                    <stddev>0.01</stddev>
                 </noise>
-            </lidar>
-        </sensor>
-    </gazebo>
-    <gazebo reference="imu_link">
-        <sensor name="imu" type="imu">
-            <always_on>1</always_on>
-            <update_rate>100</update_rate>
-            <visualize>true</visualize>
-            <topic>imu</topic>
-            <enable_metrics>true</enable_metrics>
-        </sensor>
-    </gazebo>
-<gazebo reference="laser_link">
-        <sensor name="laser_link" type="gpu_lidar">
-            <topic>scan</topic>
-            <update_rate>15</update_rate>
-            <alwaysOn>1</alwaysOn>
-            <visualize>true</visualize>
-            <lidar>
+            </ray>
+            <plugin name="laser" filename="libgazebo_ros_ray_sensor.so">
+                <ros>
+                    <remapping>~/out:=scan</remapping>
+                </ros>
+                <frame_name>laser_link</frame_name>
+                <output_type>sensor_msgs/LaserScan</output_type>
+            </plugin>
+        </sensor>
+    </gazebo>
+    <gazebo reference="l_sonar_sensor">
+        <sensor name="l_sonar_sensor" type="ray">
+            <pose>0 0 0 0 0 0</pose>
+            <always_on>1</always_on>
+            <update_rate>10</update_rate>
+            <visualize>true</visualize>
+            <ray>
                 <scan>
                     <horizontal>
-                        <samples>640</samples>
-                        <resolution>1</resolution>
-                        <min_angle>${-110/180*pi}</min_angle>
-                        <max_angle>${110/180*pi}</max_angle>
+                        <samples>10</samples>
+                        <resolution>1.0</resolution>
+                        <min_angle>-0.1745</min_angle>
+                        <max_angle>0.1745</max_angle>
                     </horizontal>
                     <vertical>
-                        <samples>1</samples>
-                        <resolution>0.01</resolution>
-                        <min_angle>0</min_angle>
-                        <max_angle>0</max_angle>
+                        <samples>10</samples>
+                        <resolution>1.0</resolution>
+                        <min_angle>-0.1745</min_angle>
+                        <max_angle>0.1745</max_angle>
                     </vertical>
                 </scan>
                 <range>
-                    <min>0.08</min>
-                    <max>15.0</max>
-                    <resolution>0.01</resolution>
+                    <min>0.05</min>
+                    <max>2.0</max>
                 </range>
+            </ray>
+            <plugin name="l_sonar_sensor_plugin" filename="libgazebo_ros_ray_sensor.so">
+                <ros>
+                    <argument>~/out:=l_sonar/range</argument>
+                </ros>
+                <frame_name>l_sonar_sensor</frame_name>
+                <output_type>sensor_msgs/Range</output_type>
+            </plugin>
+        </sensor>
+    </gazebo>
+    <gazebo reference="r_sonar_sensor">
+        <sensor name="r_sonar_sensor" type="ray">
+            <pose>0 0 0 0 0 0</pose>
+            <always_on>1</always_on>
+            <update_rate>10</update_rate>
+            <visualize>true</visualize>
+            <ray>
+                <scan>
+                    <horizontal>
+                        <samples>10</samples>
+                        <resolution>1.0</resolution>
+                        <min_angle>-0.1745</min_angle>
+                        <max_angle>0.1745</max_angle>
+                    </horizontal>
+                    <vertical>
+                        <samples>10</samples>
+                        <resolution>1.0</resolution>
+                        <min_angle>-0.1745</min_angle>
+                        <max_angle>0.1745</max_angle>
+                    </vertical>
+                </scan>
+                <range>
+                    <min>0.05</min>
+                    <max>2.0</max>
+                </range>
+            </ray>
+            <plugin name="r_sonar_sensor_plugin" filename="libgazebo_ros_ray_sensor.so">
+                <ros>
+                    <argument>~/out:=r_sonar/range</argument>
+                </ros>
+                <frame_name>r_sonar_sensor</frame_name>
+                <output_type>sensor_msgs/Range</output_type>
+            </plugin>
+        </sensor>
+    </gazebo>
+    <gazebo reference="imu_link">
+        <sensor name="imu" type="imu">
+            <always_on>1</always_on>
+            <update_rate>100</update_rate>
+            <plugin name="ros_imu_sensor_plugin" filename="libgazebo_ros_imu_sensor.so">
+                <ros>
+                    <remapping>~/out:=imu</remapping>
+                </ros>
+                <frame_name>imu_link</frame_name>
+            </plugin>
+        </sensor>
+    </gazebo>
+    <gazebo reference="camera_link">
+        <sensor type="depth" name="camera">
+            <pose>0 0 0 0 0 0</pose>
+            <update_rate>30</update_rate>
+            <visualize>true</visualize>
+            <camera>
+                <horizontal_fov>1.2113</horizontal_fov>
+                <image>
+                    <width>640</width>
+                    <height>480</height>
+                    <format>B8G8R8</format>
+                </image>
+                <depth_camera>
+                </depth_camera>
+                <clip>
+                    <near>0.02</near>
+                    <far>300</far>
+                </clip>
                 <noise>
                     <type>gaussian</type>
@@ -131,65 +191,29 @@
                     <stddev>0.02</stddev>
                 </noise>
-            </lidar>
-        </sensor>
-    </gazebo>
-    <gazebo reference="imu_link">
-        <sensor name="imu" type="imu">
-            <always_on>1</always_on>
-            <update_rate>100</update_rate>
-            <visualize>true</visualize>
-            <topic>imu</topic>
-            <enable_metrics>true</enable_metrics>
-        </sensor>
-    </gazebo>
-    <gazebo reference="camera_link">
-        <sensor name="rgbd_camera" type="rgbd_camera">
-            <always_on>1</always_on>
-            <update_rate>30</update_rate>
-            <visualize>true</visualize>
-            <topic>camera</topic>
-            <enable_metrics>true</enable_metrics>
-            <camera>
-                <horizontal_fov>1.047</horizontal_fov>
-                <image>
-                    <width>640</width>
-                    <height>480</height>
-                </image>
-                <clip>
-                    <near>0.1</near>
-                    <far>100</far>
-                </clip>
             </camera>
-            <noise>
-                <type>gaussian</type>
-                <mean>0.0</mean>
-                <stddev>0.02</stddev>
-            </noise>
-        </sensor>
-    </gazebo>
-    <gazebo reference="camera_link">
-        <sensor name="rgbd_camera" type="rgbd_camera">
-            <always_on>1</always_on>
-            <update_rate>30</update_rate>
-            <visualize>true</visualize>
-            <topic>camera</topic>
-            <enable_metrics>true</enable_metrics>
-            <camera>
-                <horizontal_fov>1.047</horizontal_fov>
-                <image>
-                    <width>640</width>
-                    <height>480</height>
-                </image>
-                <clip>
-                    <near>0.1</near>
-                    <far>100</far>
-                </clip>
-            </camera>
-            <noise>
-                <type>gaussian</type>
-                <mean>0.0</mean>
-                <stddev>0.02</stddev>
-            </noise>
-        </sensor>
-    </gazebo> -->
+            <plugin name="camera_controller" filename="libgazebo_ros_camera.so">
+                <ros>
+                </ros>
+                <baseline>0.2</baseline>
+                <alwaysOn>true</alwaysOn>
+                <updateRate>0.0</updateRate>
+                <camera_name>camera</camera_name>
+                <frame_name>camera_depth_frame</frame_name>
+                <pointCloudCutoff>0.5</pointCloudCutoff>
+                <pointCloudCutoffMax>3.0</pointCloudCutoffMax>
+                <distortionK1>0</distortionK1>
+                <distortionK2>0</distortionK2>
+                <distortionK3>0</distortionK3>
+                <distortionT1>0</distortionT1>
+                <distortionT2>0</distortionT2>
+                <CxPrime>0</CxPrime>
+                <Cx>0</Cx>
+                <Cy>0</Cy>
+                <focalLength>0</focalLength>
+                <hackBaseline>0</hackBaseline>
+                <min_depth>0.1</min_depth>
+                <max_depth>10</max_depth>
+            </plugin>
+        </sensor>
+    </gazebo>
 </robot>

File: former_description/urdf/former_ros2_control.urdf.xacro (robot description, xacro)
@@ -5,5 +5,5 @@
             <xacro:if value="$(arg use_gazebo_sim)">
                 <hardware>
-                    <plugin>gz_ros2_control/GazeboSimSystem</plugin>
+                    <plugin>gazebo_ros2_control/GazeboSystem</plugin>
                 </hardware>
             </xacro:if>
