Commit message: implementation for detecting charging station

File: former_description/urdf/former.urdf.xacro (robot description, xacro)
@@ -74,5 +74,6 @@
                     <mass value="0.843041"/>
                     <!-- <xacro:cylinder_inertia m="0.843041" r="0.0845" h="0.05"/> -->
-                    <inertia ixx="0.002632" ixy="0.000000" ixz="0.000000" iyy="0.001536" iyz="0.000000" izz="0.001536"/>
+                    <!-- <inertia ixx="0.002632" ixy="0.000000" ixz="0.000000" iyy="0.001536" iyz="0.000000" izz="0.001536"/> -->
+                    <inertia ixx="1.0" ixy="0.000000" ixz="0.000000" iyy="1.0" iyz="0.000000" izz="1.0"/>
                 </inertial>
             </link>
@@ -254,5 +255,5 @@
             <parent link="${prefix}lidar_mount"/>
             <child link="${prefix}laser_link"/>
-            <origin xyz="0 0 0.060" rpy="${pi} 0 0"/>
+            <origin xyz="0 0 0.060" rpy="0 0 0"/>
         </joint>
         <xacro:sensor_d435i parent="${prefix}base_link" name="${prefix}camera" use_nominal_extrinsics="false">

File: former_description/urdf/former_gazebo.urdf.xacro (robot description, xacro)
@@ -60,12 +60,12 @@
                 <scan>
                     <horizontal>
-                        <samples>640</samples>
+                        <samples>660</samples>
                         <resolution>1</resolution>
-                        <min_angle>-1.26889</min_angle>
-                        <max_angle>1.268899</max_angle>
+                        <min_angle>${-110*pi/180}</min_angle>
+                        <max_angle>${110*pi/180}</max_angle>
                     </horizontal>
                 </scan>
                 <range>
-                    <min>0.1</min>
+                    <min>0.05</min>
                     <max>15</max>
                     <resolution>0.01</resolution>
@@ -74,5 +74,5 @@
                     <type>gaussian</type>
                     <mean>0.0</mean>
-                    <stddev>0.01</stddev>
+                    <stddev>0.005</stddev>
                 </noise>
             </ray>

Commit message: Add suspension joint for  main wheel (check needed)

File: former_description/urdf/former.urdf.xacro (robot description, xacro)
@@ -30,4 +30,30 @@
         </joint>
         <xacro:macro name="insert_wheel" params="parent prefix dir">
+            <link name="${prefix}_wheel_suspension">
+                <visual>
+                    <origin xyz="0 0 0" rpy="0 0 ${-dir*pi/2}"/>
+                    <geometry>
+                        <mesh filename="package://former_description/meshes/visual/main_wheel_suspension.dae" scale="1 1 1"/>
+                    </geometry>
+                </visual>
+                <collision>
+                    <origin xyz="0 0 0" rpy="0 0 ${-dir*pi/2}"/>
+                    <geometry>
+                        <mesh filename="package://former_description/meshes/collision/main_wheel_suspension.stl" scale="1 1 1"/>
+                    </geometry>
+                </collision>
+                <inertial>
+                    <origin xyz="0.000 ${dir*0.026} 0.003" rpy="0 0 0"/>
+                    <mass value="0.068691"/>
+                    <inertia ixx="0.000014" ixy="0.000000" ixz="0.000000" iyy="0.000054" iyz="0.000000" izz="0.000061"/>
+                </inertial>
+            </link>
+            <joint name="${prefix}_wheel_suspension_joint" type="prismatic">
+                <parent link="${parent}" />
+                <child link="${prefix}_wheel_suspension" />
+                <axis xyz="0 0 1"/>
+                <origin xyz="0 ${dir*0.0741} 0" rpy="0 0 0"/>
+                <limit effort="10" velocity="0.1" lower="-0.01" upper="0.01"/>
+            </joint>
             <link name="${prefix}_wheel_mount">
                 <visual>
@@ -44,13 +70,13 @@
                 </collision>
                 <inertial>
-                    <origin xyz="0.026 0.000 0.000" rpy="0 0 ${dir*pi/2}"/>
-                    <mass value="0.007885"/>
-                    <inertia ixx="0.000000" ixy="0.000000" ixz="0.000000" iyy="0.000002" iyz="0.000000" izz="0.000002"/>
+                    <origin xyz="0.000 ${dir*0.026} 0.000" rpy="0 0 0"/>
+                    <mass value="0.07885"/>
+                    <inertia ixx="0.000002" ixy="0.000000" ixz="0.000000" iyy="0.0000003" iyz="0.000000" izz="0.000002"/>
                 </inertial>
             </link>
             <joint name="${prefix}_wheel_mount_fixed" type="fixed">
-                <parent link="${parent}"/>
+                <parent link="${prefix}_wheel_suspension"/>
                 <child link="${prefix}_wheel_mount"/>
-                <origin xyz="0 ${dir*0.0711} 0" rpy="0 0 0"/>
+                <origin xyz="0 ${dir*-0.003} 0" rpy="0 0 0"/>
             </joint>
             <link name="${prefix}_wheel">
@@ -62,18 +88,14 @@
                 </visual>
                 <collision>
-                    <!-- <origin xyz="0 ${dir*0.025} 0" rpy="${dir*pi/2} 0 0"/> -->
-                    <origin xyz="0 0 0" rpy="0 0 ${dir*pi/2}"/>
-                    <geometry>
-                        <!-- <cylinder radius="0.0845" length="0.05"/> -->
+                    <origin xyz="0 0 0" rpy="0 0 ${dir*pi/2}"/>
+                    <geometry>
                         <mesh filename="package://former_description/meshes/collision/main_wheel.stl" scale="1 1 1"/>
                     </geometry>
                 </collision>
                 <inertial>
-                    <!-- <origin xyz="0 ${dir*0.025} 0" rpy="${dir*pi/2} 0 0"/> -->
-                    <origin xyz="0.000 ${dir*0.031} 0.000" rpy="0 0 ${dir*pi/2}"/>
+                    <origin xyz="${dir*0.031} 0.000 0.000" rpy="0 0 0"/>
                     <mass value="0.843041"/>
-                    <!-- <xacro:cylinder_inertia m="0.843041" r="0.0845" h="0.05"/> -->
                     <!-- <inertia ixx="0.002632" ixy="0.000000" ixz="0.000000" iyy="0.001536" iyz="0.000000" izz="0.001536"/> -->
-                    <inertia ixx="1.0" ixy="0.000000" ixz="0.000000" iyy="1.0" iyz="0.000000" izz="1.0"/>
+                    <inertia ixx="0.1" ixy="0.0" ixz="0.0" iyy="0.1" iyz="0.0" izz="0.1"/>
                 </inertial>
             </link>

File: former_description/urdf/former_gazebo.urdf.xacro (robot description, xacro)
@@ -47,4 +47,26 @@
         <kd>1.0</kd>
         <!-- <minDepth>0.001</minDepth> -->
+    </gazebo>
+    <gazebo reference="l_wheel_suspension_joint">
+        <dynamics>
+            <spring_stiffness>10</spring_stiffness>
+            <spring_reference>0.06</spring_reference>
+            <damping>10.0</damping>
+            <friction>0.75</friction>
+        </dynamics>
+    </gazebo>
+    <gazebo reference="r_wheel_suspension_joint">
+        <dynamics>
+            <spring_stiffness>10</spring_stiffness>
+            <spring_reference>0.06</spring_reference>
+            <damping>10.0</damping>
+            <friction>0.75</friction>
+        </dynamics>
+    </gazebo>
+    <gazebo reference="l_wheel">
+        <self_collide>0</self_collide>
+    </gazebo>
+    <gazebo reference="r_wheel">
+        <self_collide>0</self_collide>
     </gazebo>
     <gazebo reference="base_footprint">
@@ -114,5 +136,5 @@
             <plugin name="l_sonar_sensor_plugin" filename="libgazebo_ros_ray_sensor.so">
                 <ros>
-                    <argument>~/out:=l_sonar/range</argument>
+                    <remapping>~/out:=l_sonar/range</remapping>
                 </ros>
                 <frame_name>l_sonar_sensor</frame_name>
@@ -149,5 +171,5 @@
             <plugin name="r_sonar_sensor_plugin" filename="libgazebo_ros_ray_sensor.so">
                 <ros>
-                    <argument>~/out:=r_sonar/range</argument>
+                    <remapping>~/out:=r_sonar/range</remapping>
                 </ros>
                 <frame_name>r_sonar_sensor</frame_name>
@@ -158,10 +180,66 @@
     <gazebo reference="imu_link">
         <sensor name="imu" type="imu">
-            <always_on>1</always_on>
+            <always_on>true</always_on>
             <update_rate>100</update_rate>
+            <visualize>true</visualize>
+            <imu>
+                <angular_velocity>
+                    <x>
+                        <noise type="gaussian">
+                            <mean>0.0</mean>
+                            <stddev>2e-4</stddev>
+                            <bias_mean>0.0000075</bias_mean>
+                            <bias_stddev>0.0000008</bias_stddev>
+                        </noise>
+                    </x>
+                    <y>
+                        <noise type="gaussian">
+                            <mean>0.0</mean>
+                            <stddev>2e-4</stddev>
+                            <bias_mean>0.0000075</bias_mean>
+                            <bias_stddev>0.0000008</bias_stddev>
+                        </noise>
+                    </y>
+                    <z>
+                        <noise type="gaussian">
+                            <mean>0.0</mean>
+                            <stddev>2e-4</stddev>
+                            <bias_mean>0.0000075</bias_mean>
+                            <bias_stddev>0.0000008</bias_stddev>
+                        </noise>
+                    </z>
+                </angular_velocity>
+                <linear_acceleration>
+                    <x>
+                        <noise type="gaussian">
+                            <mean>0.0</mean>
+                            <stddev>1.7e-2</stddev>
+                            <bias_mean>0.1</bias_mean>
+                            <bias_stddev>0.001</bias_stddev>
+                        </noise>
+                    </x>
+                    <y>
+                        <noise type="gaussian">
+                            <mean>0.0</mean>
+                            <stddev>1.7e-2</stddev>
+                            <bias_mean>0.1</bias_mean>
+                            <bias_stddev>0.001</bias_stddev>
+                        </noise>
+                    </y>
+                    <z>
+                        <noise type="gaussian">
+                            <mean>0.0</mean>
+                            <stddev>1.7e-2</stddev>
+                            <bias_mean>0.1</bias_mean>
+                            <bias_stddev>0.001</bias_stddev>
+                        </noise>
+                    </z>
+                </linear_acceleration>
+            </imu>
             <plugin name="ros_imu_sensor_plugin" filename="libgazebo_ros_imu_sensor.so">
                 <ros>
                     <remapping>~/out:=imu</remapping>
                 </ros>
+                <initial_orientation_as_reference>false</initial_orientation_as_reference>
                 <frame_name>imu_link</frame_name>
             </plugin>

Commit message: Add package navigation2 for former robot

File: former_description/urdf/former.urdf.xacro (robot description, xacro)
@@ -49,10 +49,10 @@
                 </inertial>
             </link>
-            <joint name="${prefix}_wheel_suspension_joint" type="prismatic">
+            <joint name="${prefix}_wheel_suspension_joint" type="fixed">
                 <parent link="${parent}" />
                 <child link="${prefix}_wheel_suspension" />
-                <axis xyz="0 0 1"/>
+                <!-- <axis xyz="0 0 1"/> -->
                 <origin xyz="0 ${dir*0.0741} 0" rpy="0 0 0"/>
-                <limit effort="10" velocity="0.1" lower="-0.01" upper="0.01"/>
+                <!-- <limit effort="10" velocity="0.1" lower="-0.01" upper="0.01"/> -->
             </joint>
             <link name="${prefix}_wheel_mount">

Commit message: add realsense2

File: former_description/urdf/former.urdf.xacro (robot description, xacro)
@@ -280,12 +280,12 @@
         </joint>
         <xacro:sensor_d435i parent="${prefix}base_link" name="${prefix}camera" use_nominal_extrinsics="false">
-            <origin xyz="0.1777 0 0.06715" rpy="0 ${-15*pi/180} 0"/>
+            <origin xyz="0.1777 0 0.06715" rpy="0 ${-12.5*pi/180} 0"/>
         </xacro:sensor_d435i>
-        <link name="${prefix}camera_depth_frame"/>
+        <!-- <link name="${prefix}camera_depth_frame"/>
         <joint name="${prefix}camera_depth_frame_fixed" type="fixed">
             <parent link="${prefix}camera_link"/>
             <child link="${prefix}camera_depth_frame"/>
             <origin xyz="0 0 0" rpy="${-pi/2} 0 ${-pi/2}"/>
-        </joint>
+        </joint> -->
     </xacro:macro>
 </robot>

Commit message: bug fixed

File: former_description/urdf/former.urdf.xacro (robot description, xacro)
@@ -280,5 +280,5 @@
         </joint>
         <xacro:sensor_d435i parent="${prefix}base_link" name="${prefix}camera" use_nominal_extrinsics="false">
-            <origin xyz="0.1777 0 0.06715" rpy="0 ${-12.5*pi/180} 0"/>
+            <origin xyz="0.1777 0 0.06715" rpy="0 ${-15*pi/180} 0"/>
         </xacro:sensor_d435i>
         <!-- <link name="${prefix}camera_depth_frame"/>
