Commit message: Support Ignition Gazebo

File: former_description/urdf/former.urdf.xacro (robot description, xacro)
@@ -90,5 +90,6 @@
                     <origin xyz="0 0 0" rpy="0 0 ${dir*pi/2}"/>
                     <geometry>
-                        <mesh filename="package://former_description/meshes/collision/main_wheel.stl" scale="1 1 1"/>
+                        <!-- <mesh filename="package://former_description/meshes/collision/main_wheel.stl" scale="1 1 1"/> -->
+                        <sphere radius="0.0845"/>
                     </geometry>
                 </collision>
@@ -105,4 +106,5 @@
                 <axis xyz="0 1 0"/>
                 <origin xyz="0 ${dir*0.051} 0" rpy="0 0 0"/>
+                <dynamics damping="0.2"/>
             </joint>
         </xacro:macro>

File: former_description/urdf/former_gazebo.urdf.xacro (robot description, xacro)
@@ -2,6 +2,13 @@
 <robot xmlns:xacro="http://www.ros.org/wiki/xacro">
     <gazebo>
-        <plugin filename="libgazebo_ros2_control.so" name="gazebo_ros2_control">
-        <parameters>$(find former_bringup)/config/controllers_former_gazebo.yaml</parameters>
+        <plugin filename="ign_ros2_control-system" name="ign_ros2_control::IgnitionROS2ControlPlugin">
+            <parameters>$(find former_bringup)/config/controllers_former_gazebo.yaml</parameters>
+        </plugin>
+        <plugin filename="ignition-gazebo-sensors-system" name="gz::sim::systems::Sensors">
+            <render_engine>ogre2</render_engine>
+        </plugin>
+        <plugin filename="ignition-gazebo-imu-system" name="gz::sim::systems::Imu">
+        </plugin>
+        <plugin filename="ignition-gazebo-scene-broadcaster-system" name="gz::sim::systems::SceneBroadcaster">
         </plugin>
     </gazebo>
@@ -48,20 +55,4 @@
         <!-- <minDepth>0.001</minDepth> -->
     </gazebo>
-    <gazebo reference="l_wheel_suspension_joint">
-        <dynamics>
-            <spring_stiffness>10</spring_stiffness>
-            <spring_reference>0.06</spring_reference>
-            <damping>10.0</damping>
-            <friction>0.75</friction>
-        </dynamics>
-    </gazebo>
-    <gazebo reference="r_wheel_suspension_joint">
-        <dynamics>
-            <spring_stiffness>10</spring_stiffness>
-            <spring_reference>0.06</spring_reference>
-            <damping>10.0</damping>
-            <friction>0.75</friction>
-        </dynamics>
-    </gazebo>
     <gazebo reference="l_wheel">
         <self_collide>0</self_collide>
@@ -74,21 +65,25 @@
     </gazebo>
     <gazebo reference="laser_link">
-        <sensor name="laser" type="ray">
-            <pose>0 0 0 0 0 0</pose>
-            <always_on>1</always_on>
+        <sensor name='gpu_lidar' type='gpu_lidar'>
+            <topic>scan</topic>
             <update_rate>15</update_rate>
-            <visualize>true</visualize>
-            <ray>
+            <lidar>
                 <scan>
                     <horizontal>
-                        <samples>660</samples>
+                        <samples>640</samples>
                         <resolution>1</resolution>
-                        <min_angle>${-110*pi/180}</min_angle>
-                        <max_angle>${110*pi/180}</max_angle>
+                        <min_angle>-1.85</min_angle>
+                        <max_angle>1.85</max_angle>
                     </horizontal>
+                    <vertical>
+                        <samples>1</samples>
+                        <resolution>0.01</resolution>
+                        <min_angle>0</min_angle>
+                        <max_angle>0</max_angle>
+                    </vertical>
                 </scan>
                 <range>
-                    <min>0.05</min>
-                    <max>15</max>
+                    <min>0.08</min>
+                    <max>15.0</max>
                     <resolution>0.01</resolution>
                 </range>
@@ -96,16 +91,12 @@
                     <type>gaussian</type>
                     <mean>0.0</mean>
-                    <stddev>0.005</stddev>
+                    <stddev>0.01</stddev>
                 </noise>
-            </ray>
-            <plugin name="laser" filename="libgazebo_ros_ray_sensor.so">
-                <ros>
-                    <remapping>~/out:=scan</remapping>
-                </ros>
-                <frame_name>laser_link</frame_name>
-                <output_type>sensor_msgs/LaserScan</output_type>
-            </plugin>
-        </sensor>
-    </gazebo>
+            </lidar>
+            <alwaysOn>1</alwaysOn>
+            <visualize>true</visualize>
+        </sensor>
+    </gazebo>
+    <!--
     <gazebo reference="l_sonar_sensor">
         <sensor name="l_sonar_sensor" type="ray">
@@ -178,9 +169,12 @@
         </sensor>
     </gazebo>
+    -->
     <gazebo reference="imu_link">
         <sensor name="imu" type="imu">
-            <always_on>true</always_on>
+            <always_on>1</always_on>
             <update_rate>100</update_rate>
             <visualize>true</visualize>
+            <topic>imu_raw</topic>
+            <enable_metrics>true</enable_metrics>
             <imu>
                 <angular_velocity>
@@ -237,18 +231,8 @@
                 </linear_acceleration>
             </imu>
-            <plugin name="ros_imu_sensor_plugin" filename="libgazebo_ros_imu_sensor.so">
-                <ros>
-                    <remapping>~/out:=imu</remapping>
-                </ros>
-                <initial_orientation_as_reference>false</initial_orientation_as_reference>
-                <frame_name>imu_link</frame_name>
-            </plugin>
         </sensor>
     </gazebo>
     <gazebo reference="camera_link">
-        <sensor type="depth" name="camera">
-            <pose>0 0 0 0 0 0</pose>
-            <update_rate>30</update_rate>
-            <visualize>true</visualize>
+        <sensor name="rgbd_camera" type="rgbd_camera">
             <camera>
                 <horizontal_fov>1.2113</horizontal_fov>
@@ -256,11 +240,8 @@
                     <width>640</width>
                     <height>480</height>
-                    <format>B8G8R8</format>
                 </image>
-                <depth_camera>
-                </depth_camera>
                 <clip>
-                    <near>0.02</near>
-                    <far>300</far>
+                    <near>0.1</near>
+                    <far>100</far>
                 </clip>
                 <noise>
@@ -270,27 +251,9 @@
                 </noise>
             </camera>
-            <plugin name="camera_controller" filename="libgazebo_ros_camera.so">
-                <ros>
-                </ros>
-                <baseline>0.2</baseline>
-                <alwaysOn>true</alwaysOn>
-                <updateRate>0.0</updateRate>
-                <camera_name>camera</camera_name>
-                <frame_name>camera_depth_frame</frame_name>
-                <pointCloudCutoff>0.5</pointCloudCutoff>
-                <pointCloudCutoffMax>3.0</pointCloudCutoffMax>
-                <distortionK1>0</distortionK1>
-                <distortionK2>0</distortionK2>
-                <distortionK3>0</distortionK3>
-                <distortionT1>0</distortionT1>
-                <distortionT2>0</distortionT2>
-                <CxPrime>0</CxPrime>
-                <Cx>0</Cx>
-                <Cy>0</Cy>
-                <focalLength>0</focalLength>
-                <hackBaseline>0</hackBaseline>
-                <min_depth>0.1</min_depth>
-                <max_depth>10</max_depth>
-            </plugin>
+            <always_on>1</always_on>
+            <update_rate>30</update_rate>
+            <visualize>true</visualize>
+            <topic>camera</topic>
+            <enable_metrics>true</enable_metrics>
         </sensor>
     </gazebo>

File: former_description/urdf/former_ros2_control.urdf.xacro (robot description, xacro)
@@ -5,5 +5,5 @@
             <xacro:if value="$(arg use_gazebo_sim)">
                 <hardware>
-                    <plugin>gazebo_ros2_control/GazeboSystem</plugin>
+                    <plugin>ign_ros2_control/IgnitionSystem</plugin>
                 </hardware>
             </xacro:if>
@@ -19,31 +19,33 @@
             <joint name="l_wheel_joint">
                 <command_interface name="velocity">
-                    <param name="min">-1.0</param>
-                    <param name="max">1.0</param>
+                    <param name="min">-1</param>
+                    <param name="max">1</param>
                 </command_interface>
                 <state_interface name="position"/>
                 <state_interface name="velocity"/>
-                <state_interface name="effort"/>
+                <!-- <state_interface name="effort"/> -->
             </joint>
             <joint name="r_wheel_joint">
                 <command_interface name="velocity">
-                    <param name="min">-1.0</param>
-                    <param name="max">1.0</param>
+                    <param name="min">-1</param>
+                    <param name="max">1</param>
                 </command_interface>
                 <state_interface name="position"/>
                 <state_interface name="velocity"/>
-                <state_interface name="effort"/>
+                <!-- <state_interface name="effort"/> -->
             </joint>
-            <gpio name="gpio">
-                <command_interface name="set_enable_motor"/>
-                <state_interface name="motor_enabled"/>
-                <state_interface name="estop_button_state"/>
-                <state_interface name="system_voltage"/>
-                <state_interface name="charging_voltage"/>
-                <state_interface name="user_power_current1"/>
-                <state_interface name="user_power_current2"/>
-                <state_interface name="curent_temperature"/>
-                <state_interface name="fault_flags"/>
-            </gpio>
+            <xacro:unless value="$(arg use_gazebo_sim)">
+                <gpio name="gpio">
+                    <command_interface name="set_enable_motor"/>
+                    <state_interface name="motor_enabled"/>
+                    <state_interface name="estop_button_state"/>
+                    <state_interface name="system_voltage"/>
+                    <state_interface name="charging_voltage"/>
+                    <state_interface name="user_power_current1"/>
+                    <state_interface name="user_power_current2"/>
+                    <state_interface name="curent_temperature"/>
+                    <state_interface name="fault_flags"/>
+                </gpio>
+            </xacro:unless>
         </ros2_control>
     </xacro:macro>

Commit message: 2d lidar tf modify from org source

File: former_description/urdf/former.urdf.xacro (robot description, xacro)
@@ -275,10 +275,10 @@
             <origin xyz="0.160 0 0.2275" rpy="${pi} 0 0"/>
         </joint>
-        <link name="${prefix}laser_link"/>
+        <!--link name="${prefix}laser_link"/>
         <joint name="${prefix}laser_link_fixed_joint" type="fixed">
             <parent link="${prefix}lidar_mount"/>
             <child link="${prefix}laser_link"/>
             <origin xyz="0 0 0.060" rpy="0 0 0"/>
-        </joint>
+        </joint> -->
         <xacro:sensor_d435i parent="${prefix}base_link" name="${prefix}camera" use_nominal_extrinsics="false">
             <origin xyz="0.1777 0 0.06715" rpy="0 ${-15*pi/180} 0"/>
